File: ftdi.kicad_sch (KiCad schematic)
At the start: 47 parts, among them P10 PLUG-6-PIN, P11 PLUG-6-PIN, Q1 NPN, U1 93LC46, U11 74LVC1GU04, U2 FT2232H, U3 N25Q128, X1 USBMINI, X2 12MHz

Commit message: pcb/schematic update v0.1.4
Parts:
- C1, C10, C11, C12, C13, C14, C15, C2, C3, C4, C5, C7, C8: Manufacturer (none) -> Murata Electronics; Manufacturer# (none) -> GRM033R61A104KE15D; Supplier (none) -> DigiKey
- C6, C9: Manufacturer (none) -> Cal-Chip Electronics Inc.; Manufacturer# (none) -> CHV0603N250200GCT; Supplier (none) -> DigiKey
- L1, L2: Manufacturer (none) -> Tayo Yuden; Manufacturer# (none) -> LSQBB160808T100K; Supplier (none) -> Mouser
- P10, P11: Manufacturer (none) -> Oupiin; Manufacturer# (none) -> 2011-2X03G00SB; Supplier (none) -> DigiKey
- Q1: Manufacturer (none) -> Micro Commercial Co; Manufacturer# (none) -> MMBT3904-TP
- R1, R10, R11, R13: Manufacturer (none) -> Panasonic Electronic Componenets; Manufacturer# (none) -> ERJ-1GNF1002C; Supplier (none) -> DigiKey
- R12, R4, R8, R9: Manufacturer (none) -> Panasonic Electronic Componenets; Manufacturer# (none) -> ERJ-1GN0R00C; Supplier (none) -> DigiKey
- R2: Manufacturer (none) -> Panasonic Electronic Componenets; Manufacturer# (none) -> ERJ-1GNF2201C; Supplier (none) -> DigiKey
- R3, R30, R37, R38: Manufacturer (none) -> n/a; Manufacturer# (none) -> n/a; Supplier (none) -> n/a; now not fitted; now left out of the parts list
- R35, R36, R7: Manufacturer (none) -> Panasonic Electronic Componenets; Manufacturer# (none) -> ERJ-3GEYJ103V; Supplier (none) -> DigiKey
- R39: Manufacturer (none) -> Yageo; Manufacturer# (none) -> SR0603KR-7W2K2L; Supplier (none) -> DigiKey
- R5: Manufacturer (none) -> Panasonic Electronic Componenets; Manufacturer# (none) -> ERJ-3EKF1202V; Supplier (none) -> DigiKey
- R6: Manufacturer (none) -> Panasonic Electronic Componenets; Manufacturer# (none) -> ERJ-3GEYJ472V; Supplier (none) -> DigiKey
- U1: Manufacturer (none) -> Microchip Technology; Manufacturer# (none) -> 93LC46CT-I/SN; Supplier (none) -> DigiKey
- U11: Manufacturer (none) -> Nexperia USA Inc.; Manufacturer# (none) -> 74LVC1GU04GW,125; Supplier (none) -> DigiKey
- U2: Manufacturer (none) -> FTDI; Manufacturer# (none) -> FT2232HL-REEL; Supplier (none) -> DigiKey
- U3: Manufacturer (none) -> Micron Technology Inc.; Manufacturer# (none) -> N25Q128A13ESE40G; Supplier (none) -> DigiKey
- VR1, VR2: Manufacturer (none) -> Bourns Inc.; Manufacturer# (none) -> 3361P-1-203GLF; Supplier (none) -> DigiKey
- X1: Manufacturer (none) -> Adam Tech; Manufacturer# (none) -> MUSB-B5-S-VT-TSMT-T/R; Supplier (none) -> DigiKey
- X2: Manufacturer (none) -> ECS Inc.; Manufacturer# (none) -> ECS-120-18-23A-EN-TR; Supplier (none) -> DigiKey
