File: gpios.kicad_sch (KiCad schematic)
At the start: 8 parts

Commit message: pcb/schematic update v0.1.4
Parts:
- H0, H1, H2, H3, H4, H5, H6, H7: Manufacturer (none) -> Oupiin; Manufacturer# (none) -> 2011-2X12G00SB; Supplier (none) -> DigiKey
