File: power.kicad_sch (KiCad schematic)
At the start: 18 parts, among them J1 DC_barrel, K1 VBUS_VCCIN, U6 LM1117-ADJ, U7 LM1117-ADJ, U8 LM1117-ADJ

Commit message: pcb/schematic update v0.1.4
Parts:
- C65: footprint saturn:CP_Elec_6.3x7.7 -> saturn:C_Elec_6.6x6.6; Manufacturer (none) -> KEMET; Manufacturer# (none) -> EEV476M035S9GAA; Supplier (none) -> DigiKey
- C69, C70, C71: footprint saturn:C_0201_0603Metric -> saturn:C_0402_1005Metric; Manufacturer (none) -> Murata Electronics; Manufacturer# (none) -> GRM155R60J106ME15D; Supplier (none) -> DigiKey
- C72, C73, C74: Manufacturer (none) -> Murata Electronics; Manufacturer# (none) -> GRM033R61A104KE15D; Supplier (none) -> DigiKey
- J1: Manufacturer (none) -> CUI Devices; Manufacturer# (none) -> PJ-036AH-SMT-TR; Supplier (none) -> DigiKey
- K1: Manufacturer (none) -> Oupiin; Manufacturer# (none) -> 2111-1X03G00SB; Supplier (none) -> DigiKey
- R20: Manufacturer (none) -> Panasonic Electronic Componenets; Manufacturer# (none) -> ERJ-1GNF3300C; Supplier (none) -> DigiKey
- R21: Manufacturer (none) -> Panasonic Electronic Componenets; Manufacturer# (none) -> ERJ-1GN0R00C; Supplier (none) -> DigiKey
- R22: Manufacturer (none) -> Panasonic Electronic Componenets; Manufacturer# (none) -> ERJ-1GNF1000C; Supplier (none) -> DigiKey
- R23, R24, R25: Manufacturer (none) -> Panasonic Electronic Componenets; Manufacturer# (none) -> ERJ-1GNJ221C; Supplier (none) -> DigiKey
- U6, U7, U8: Manufacturer (none) -> Texas Instruments; Manufacturer# (none) -> LM1117IMPX-ADJ/NOPB; Supplier (none) -> DigiKey
