File: ram.kicad_sch (KiCad schematic)
At the start: 13 parts, among them U9 MT46H32M16LF

Commit message: spartan6 pcb v0.1.2 -- reroute pcb and modify BGA and DDR fanouts
Parts:
- U9: footprint saturn:VFBGA60 -> saturn:MT46H32M16LF
Changed lines of the file:
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@@
     (property "Reference" "U9" (id 0) (at 146.05 44.45 0))
     (property "Value" "MT46H32M16LF" (id 1) (at 146.05 46.99 0))
-    (property "Footprint" "saturn:VFBGA60" (id 2) (at 146.05 73.66 0)
+    (property "Footprint" "saturn:MT46H32M16LF" (id 2) (at 146.05 73.66 0)
       (effects (font (size 1.27 1.27)) hide)
     )

Commit message: pcb/schematic update v0.1.4
Parts:
- C75, C76, C77, C78, C79, C80, C81, C82: Manufacturer (none) -> Murata Electronics; Manufacturer# (none) -> GRM033R61A104KE15D; Supplier (none) -> DigiKey
- R26, R27: Manufacturer (none) -> Panasonic Electronic Componenets; Manufacturer# (none) -> ERJ-1GNF1000C; Supplier (none) -> DigiKey
- R28: Manufacturer (none) -> Panasonic Electronic Componenets; Manufacturer# (none) -> ERJ-1GNF4701C; Supplier (none) -> DigiKey
- R29: Manufacturer (none) -> Stackpole Electronics Inc; Manufacturer# (none) -> RMCF0603FT100R; Supplier (none) -> DigiKey
- U9: Manufacturer (none) -> Micron Technology Inc.; Manufacturer# (none) -> MT46H32M16LFBF-5 IT:C; Supplier (none) -> DigiKey
