File: spartan6.kicad_sch (KiCad schematic)
At the start: 67 parts, among them P1 JTAG-14PIN, U10 FXO-HC536R, U4 FXO-HC536R, U5 SPARTAN6-CSG324

Commit message: spartan6 pcb v0.1.2 -- reroute pcb and modify BGA and DDR fanouts
Parts:
- R16: footprint saturn:R_0201_0603Metric -> saturn:R_0603_1608Metric
Connections:
- no-connect marks 20 -> 21
Changed lines of the file:
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@@
   (no_connect (at 294.64 41.91))
   (no_connect (at 294.64 156.21))
+  (no_connect (at 135.89 105.41))
   (bus_entry (at 229.87 118.11) (size -2.54 -2.54)
     (stroke (width 0) (type default) (color 0 0 0 0))
@@
     (stroke (width 0) (type default) (color 0 0 0 0))
   )
-  (wire (pts (xy 127 105.41) (xy 134.62 105.41))
+  (wire (pts (xy 127 105.41) (xy 135.89 105.41))
     (stroke (width 0) (type default) (color 0 0 0 0))
   )
@@
     (property "Reference" "R16" (id 0) (at 102.87 214.63 90))
     (property "Value" "10K" (id 1) (at 105.41 214.63 90))
-    (property "Footprint" "saturn:R_0201_0603Metric" (id 2) (at 107.188 214.63 90)
+    (property "Footprint" "saturn:R_0603_1608Metric" (id 2) (at 107.188 214.63 90)
       (effects (font (size 1.27 1.27)) hide)
     )

Commit message: pcb/schematic update v0.1.4
Parts:
- C16, C17: Manufacturer (none) -> n/a; Manufacturer# (none) -> n/a; Supplier (none) -> n/a; now not fitted; now left out of the parts list
- C18, C19, C20, C21, C22, C23, C24, C25, C26, C27, C28, C29, C30, C31, C32, C33, C34, C35, C36, C37, C38, C39, C40, C41, C42, C43, C44, C45, C46, C47, C48, C49, C50, C51, C52, C53, C54, C55, C56, C57, C58, C59, C60, C63, C64, C84: Manufacturer (none) -> Murata Electronics; Manufacturer# (none) -> GRM033R71A103KA01D; Supplier (none) -> DigiKey
- C83: Manufacturer (none) -> Murata Electronics; Manufacturer# (none) -> GQM1875C2E150JB12D; Supplier (none) -> DigiKey
- D1: Manufacturer (none) -> APEM Inc.; Manufacturer# (none) -> TV01WS00100; Supplier (none) -> DigiKey
- GS5, GS6, GS7: Manufacturer (none) -> n/a; Manufacturer# (none) -> n/a; Supplier (none) -> n/a; now left out of the parts list
- P1: Manufacturer (none) -> Oupiin; Manufacturer# (none) -> 2011-2X07G00SB; Supplier (none) -> DigiKey
- R14: Manufacturer (none) -> Panasonic Electronic Componenets; Manufacturer# (none) -> ERJ-3GEYJ472V; Supplier (none) -> DigiKey
- R15, R16: Manufacturer (none) -> Panasonic Electronic Componenets; Manufacturer# (none) -> ERJ-3GEYJ103V; Supplier (none) -> DigiKey
- R17, R19: Manufacturer (none) -> Panasonic Electronic Componenets; Manufacturer# (none) -> ERJ-1GNF4701C; Supplier (none) -> DigiKey
- R18: Manufacturer (none) -> Panasonic Electronic Componenets; Manufacturer# (none) -> ERJ-3EKF1001V; Supplier (none) -> DigiKey
- R31, R32, R33, R34: Manufacturer (none) -> Stackpole Electronics Inc; Manufacturer# (none) -> RMCF0603ZT0R00; Supplier (none) -> DigiKey
- U10: Manufacturer (none) -> Renesas Electronics Corporation; Manufacturer# (none) -> XLH536100.000000I; Supplier (none) -> DigiKey
- U4: Manufacturer (none) -> Renesas Electronics Corporation; Manufacturer# (none) -> XLH536100.000000I; Supplier (none) -> DigiKey; now not fitted; now left out of the parts list
- U5: Manufacturer (none) -> AMD; Manufacturer# (none) -> XC6SLX45-2CSG324C; Supplier (none) -> DigiKey
